File: AlarmClock.brd (EAGLE design)
At the start: 100 x 80 mm, 20 parts, among them IC1 LD1117AS33TR, T1 BC848

Commit message: Add files via upload
Parts:
- R1: value (none) -> 10k
Changed lines of the file:
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@@
 <attribute name="POPULARITY" value="0" x="59" y="16" size="1.778" layer="27" rot="R270" display="off"/>
 </element>
-<element name="R1" library="rcl" library_urn="urn:adsk.eagle:library:334" package="R1206" package3d_urn="urn:adsk.eagle:package:23540/2" value="" x="58" y="22" smashed="yes" rot="R270">
+<element name="R1" library="rcl" library_urn="urn:adsk.eagle:library:334" package="R1206" package3d_urn="urn:adsk.eagle:package:23540/2" value="10k" x="58" y="22" smashed="yes" rot="R270">
 <attribute name="NAME" x="56.93" y="24.67" size="1.27" layer="25"/>
 <attribute name="SPICEPREFIX" value="R" x="58" y="22" size="1.778" layer="27" rot="R270" display="off"/>
-<attribute name="VALUE" x="55.46" y="23.27" size="1.27" layer="27" rot="R270"/>
 </element>
 <element name="JP1" library="pinhead-ext" package="1X02" value="" x="30" y="68" smashed="yes">

Commit message: Add files via upload
Parts:
- renumbered JP1 to BTN
Connections:
- net IO25: now also BME280.3
- net IO26: now also R1.1
- net IO27: now also LCD.31
- net IO32: now also BME280.4; no longer LCD.31
- net IO34: no longer BME280.3
- net IO35: now also BTN.2; no longer R1.1
- net SENSOR_VN: no longer BME280.4
- net SENSOR_VP: no longer BTN.2
Routing:
- net IO27: track 0.00 -> 80.3 mm
- net IO34: track 67.2 -> 0.00 mm
- net SENSOR_VN: track 66.9 -> 0.00 mm
- net SENSOR_VP: track 63.8 -> 0.00 mm
- net IO25: track 0.00 -> 60.4 mm
- net IO35: track 25.3 -> 61.4 mm
- net IO32: track 84.4 -> 61.4 mm
- net IO26: track 0.00 -> 20.0 mm
Changed lines of the file:
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@@
 <attribute name="SPICEPREFIX" value="R" x="58" y="22" size="1.778" layer="27" rot="R270" display="off"/>
 </element>
-<element name="JP1" library="pinhead-ext" package="1X02" value="" x="30" y="68" smashed="yes">
-<attribute name="NAME" x="27.3838" y="69.8288" size="1.27" layer="25" ratio="10"/>
+<element name="BTN" library="pinhead-ext" package="1X02" value="" x="30" y="68" smashed="yes">
+<attribute name="NAME" x="28.2838" y="69.8288" size="1.27" layer="25" ratio="10"/>
 <attribute name="VALUE" x="27.46" y="64.825" size="1.27" layer="27"/>
 </element>
@@
 <contactref element="BME280" pad="5"/>
 <contactref element="T1" pad="2"/>
-<contactref element="JP1" pad="1"/>
+<contactref element="BTN" pad="1"/>
 </signal>
 <signal name="VDD">
@@
 <wire x1="13.35" y1="63.35" x2="12" y2="62" width="0.6096" layer="1"/>
 <wire x1="12" y1="62" x2="12" y2="50" width="0.6096" layer="1"/>
-<wire x1="14" y1="48" x2="19.8516125" y2="48" width="0.6096" layer="1"/>
-<wire x1="19.8516125" y1="48" x2="54.8516125" y2="13" width="0.6096" layer="1"/>
+<wire x1="14" y1="48" x2="18.9516125" y2="48" width="0.6096" layer="1"/>
+<wire x1="18.9516125" y1="48" x2="53.9516125" y2="13" width="0.6096" layer="1"/>
 <contactref element="SG1" pad="+"/>
 <wire x1="77.51" y1="13" x2="74.81" y2="15.7" width="0.6096" layer="1"/>
 <wire x1="90.24" y1="13" x2="77.51" y2="13" width="0.6096" layer="1"/>
-<wire x1="54.8516125" y1="13" x2="72.11" y2="13" width="0.6096" layer="1"/>
+<wire x1="53.9516125" y1="13" x2="72.11" y2="13" width="0.6096" layer="1"/>
 <wire x1="72.11" y1="13" x2="74.81" y2="15.7" width="0.6096" layer="1"/>
 <wire x1="50.5" y1="71.6" x2="53.5" y2="68.6" width="0.6096" layer="1"/>
@@
 <signal name="SENSOR_VP">
 <contactref element="ESP32" pad="4"/>
-<wire x1="31.27" y1="50.93" x2="45.5" y2="36.7" width="0.508" layer="1"/>
-<wire x1="45.5" y1="36.7" x2="53.7" y2="36.7" width="0.508" layer="1"/>
-<wire x1="53.7" y1="36.7" x2="55.1" y2="38.1" width="0.508" layer="1"/>
-<wire x1="55.1" y1="38.1" x2="55.1" y2="44.4" width="0.508" layer="1"/>
-<wire x1="55.1" y1="44.4" x2="59.84" y2="49.14" width="0.508" layer="1"/>
-<wire x1="59.84" y1="49.14" x2="63.3" y2="49.14" width="0.508" layer="1"/>
-<contactref element="JP1" pad="2"/>
-<wire x1="31.27" y1="68" x2="31.27" y2="50.93" width="0.508" layer="1"/>
 </signal>
 <signal name="SENSOR_VN">
 <contactref element="ESP32" pad="5"/>
-<wire x1="42.5" y1="35" x2="53.8" y2="35" width="0.508" layer="1"/>
-<wire x1="53.8" y1="35" x2="56.3" y2="37.5" width="0.508" layer="1"/>
-<wire x1="56.3" y1="37.5" x2="56.3" y2="43.7" width="0.508" layer="1"/>
-<wire x1="56.3" y1="43.7" x2="60.47" y2="47.87" width="0.508" layer="1"/>
-<wire x1="60.47" y1="47.87" x2="63.3" y2="47.87" width="0.508" layer="1"/>
-<contactref element="BME280" pad="4"/>
-<wire x1="42.5" y1="35" x2="19.23" y2="58.27" width="0.508" layer="1"/>
-<wire x1="15" y1="58.27" x2="19.23" y2="58.27" width="0.508" layer="1"/>
 </signal>
 <signal name="IO34">
 <contactref element="ESP32" pad="6"/>
-<contactref element="BME280" pad="3"/>
-<wire x1="57.4396" y1="36.5" x2="53.9396" y2="33" width="0.508" layer="1"/>
-<wire x1="40" y1="33" x2="17.27" y2="55.73" width="0.508" layer="1"/>
-<wire x1="15" y1="55.73" x2="17.27" y2="55.73" width="0.508" layer="1"/>
-<wire x1="40" y1="33" x2="53.9396" y2="33" width="0.508" layer="1"/>
-<wire x1="63.3" y1="46.6" x2="60.9" y2="46.6" width="0.508" layer="1"/>
-<wire x1="57.4396" y1="43.1396" x2="57.4396" y2="36.5" width="0.508" layer="1"/>
-<wire x1="60.9" y1="46.6" x2="57.4396" y2="43.1396" width="0.508" layer="1"/>
 </signal>
 <signal name="IO35">
 <contactref element="ESP32" pad="7"/>
-<wire x1="63.3" y1="45.33" x2="61.33" y2="45.33" width="0.508" layer="1"/>
-<contactref element="R1" pad="1"/>
-<wire x1="58.6" y1="42.6" x2="58.6" y2="24.022" width="0.508" layer="1"/>
-<wire x1="58.6" y1="24.022" x2="58" y2="23.422" width="0.508" layer="1"/>
-<wire x1="61.33" y1="45.33" x2="58.6" y2="42.6" width="0.508" layer="1"/>
+<contactref element="BTN" pad="2"/>
+<wire x1="63.3" y1="45.33" x2="61.93" y2="45.33" width="0.508" layer="1"/>
+<wire x1="53.6" y1="37" x2="40" y2="37" width="0.508" layer="1"/>
+<wire x1="40" y1="37" x2="31.27" y2="45.73" width="0.508" layer="1"/>
+<wire x1="31.27" y1="45.73" x2="31.27" y2="68" width="0.508" layer="1"/>
+<wire x1="61.93" y1="45.33" x2="53.6" y2="37" width="0.508" layer="1"/>
 </signal>
 <signal name="IO26">
 <contactref element="ESP32" pad="11"/>
+<contactref element="R1" pad="1"/>
+<wire x1="63.3" y1="40.25" x2="61.55" y2="40.25" width="0.508" layer="1"/>
+<wire x1="61.55" y1="40.25" x2="58" y2="36.7" width="0.508" layer="1"/>
+<wire x1="58" y1="36.7" x2="58" y2="23.422" width="0.508" layer="1"/>
 </signal>
 <signal name="IO14">
@@
 <signal name="IO32">
 <contactref element="ESP32" pad="8"/>
-<contactref element="LCD" pad="31"/>
 <wire x1="63.3" y1="44.06" x2="63.24" y2="44" width="0.508" layer="1"/>
-<wire x1="63.24" y1="44" x2="62" y2="44" width="0.508" layer="1"/>
-<wire x1="62" y1="44" x2="60.1" y2="42.1" width="0.508" layer="1"/>
-<wire x1="60.1" y1="42.1" x2="60.1" y2="30.7" width="0.508" layer="1"/>
-<wire x1="60.1" y1="30.7" x2="66.3" y2="24.5" width="0.508" layer="1"/>
-<wire x1="95" y1="25.8" x2="95" y2="51" width="0.508" layer="1"/>
-<wire x1="95" y1="51" x2="93.5" y2="52.5" width="0.508" layer="1"/>
-<wire x1="91.52" y1="52.5" x2="90.31" y2="53.71" width="0.508" layer="1"/>
-<wire x1="66.3" y1="24.5" x2="93.7" y2="24.5" width="0.508" layer="1"/>
-<wire x1="93.7" y1="24.5" x2="95" y2="25.8" width="0.508" layer="1"/>
-<wire x1="93.5" y1="52.5" x2="91.52" y2="52.5" width="0.508" layer="1"/>
+<contactref element="BME280" pad="4"/>
+<wire x1="63.3" y1="44.06" x2="63.2864" y2="44.0464" width="0.508" layer="1"/>
+<wire x1="63.2864" y1="44.0464" x2="62.1816625" y2="44.0464" width="0.508" layer="1"/>
+<wire x1="62.1816625" y1="44.0464" x2="53.6352625" y2="35.5" width="0.508" layer="1"/>
+<wire x1="38.77" y1="35.5" x2="16" y2="58.27" width="0.508" layer="1"/>
+<wire x1="16" y1="58.27" x2="15" y2="58.27" width="0.508" layer="1"/>
+<wire x1="53.6352625" y1="35.5" x2="38.77" y2="35.5" width="0.508" layer="1"/>
 </signal>
 <signal name="IO33">
@@
 <signal name="IO25">
 <contactref element="ESP32" pad="10"/>
+<contactref element="BME280" pad="3"/>
+<wire x1="15" y1="55.73" x2="16.27" y2="55.73" width="0.508" layer="1"/>
+<wire x1="61.22" y1="41.52" x2="63.3" y2="41.52" width="0.508" layer="1"/>
+<wire x1="16.27" y1="55.73" x2="38" y2="34" width="0.508" layer="1"/>
+<wire x1="38" y1="34" x2="53.7" y2="34" width="0.508" layer="1"/>
+<wire x1="53.7" y1="34" x2="61.22" y2="41.52" width="0.508" layer="1"/>
 </signal>
 <signal name="N$5">
@@
 <signal name="IO27">
 <contactref element="ESP32" pad="12"/>
+<contactref element="LCD" pad="31"/>
+<wire x1="63.3" y1="38.98" x2="61.98" y2="38.98" width="0.508" layer="1"/>
+<wire x1="60" y1="37" x2="60" y2="29" width="0.508" layer="1"/>
+<wire x1="60" y1="29" x2="64.5" y2="24.5" width="0.508" layer="1"/>
+<wire x1="64.5" y1="24.5" x2="93.5" y2="24.5" width="0.508" layer="1"/>
+<wire x1="93.5" y1="24.5" x2="94.9" y2="25.9" width="0.508" layer="1"/>
+<wire x1="94.9" y1="51.1" x2="93.5" y2="52.5" width="0.508" layer="1"/>
+<wire x1="91.52" y1="52.5" x2="90.31" y2="53.71" width="0.508" layer="1"/>
+<wire x1="61.98" y1="38.98" x2="60" y2="37" width="0.508" layer="1"/>
+<wire x1="94.9" y1="25.9" x2="94.9" y2="51.1" width="0.508" layer="1"/>
+<wire x1="93.5" y1="52.5" x2="91.52" y2="52.5" width="0.508" layer="1"/>
 </signal>
 <signal name="IO23">
