File: AlarmClock.brd (EAGLE design)
At the start: 100 x 80 mm, 20 parts, among them IC1 LD1117AS33TR, T1 BC848

Commit message: Add files via upload
Parts:
- BT1, BT2, BT3: value (none) -> HALTER1XUM4-LF; device SparkFun-Batteries:BATTERY-AAA -> TheLibrary:HALTER1XUM4-LF
- moved BT1 22.0 mm to (30.0, 20.1)
- moved BT3 18.0 mm to (29.9, 48.0), turned to 180 degrees
- moved BT2 16.0 mm to (31.0, 34.0), turned to 0 degrees
- moved IC1 13.3 mm to (35.1, 60.4)
- moved BME280 9.22 mm to (9.00, 64.0)
- moved C2 7.81 mm to (58.0, 46.0), turned to 90 degrees
- moved C6 3.00 mm to (43.0, 59.0)
- moved C1 1.00 mm to (58.0, 69.0)
- moved R1 1.00 mm to (59.0, 22.0)
- moved RST 1.00 mm to (63.0, 69.0)
- moved SG1 1.00 mm to (72.0, 15.7)
- moved T1 1.00 mm to (60.0, 16.0)
- moved C3 0.10 mm to (53.0, 59.0), turned to 270 degrees
- moved C4 0.10 mm to (58.0, 59.0), turned to 270 degrees
- turned BTN to 180 degrees
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Connections:
- net GND: now also BT1.P$2; no longer BT2.GND@1
- net N$5: now also BT1.P$1, BT2.P$2; no longer BT2.PWR@1, BT3.GND@1
- net N$6: now also BT2.P$1, BT3.P$2; no longer BT1.GND@1, BT3.PWR@1
- net VIN: now also BT3.P$1; no longer BT1.PWR@1
Routing:
- net VDD: track 225.5 -> 234.3 mm
- net IO25: track 60.4 -> 65.2 mm
- net IO32: track 61.4 -> 66.0 mm
- net IO35: track 61.4 -> 58.0 mm
- net VIN: track 53.9 -> 57.1 mm
- net N$5: track 12.0 -> 14.3 mm
- net RXD0: track 61.2 -> 63.4 mm
- net TXD0: track 60.7 -> 62.7 mm
- net EN: track 10.4 -> 8.52 mm
- net IO0: track 61.3 -> 63.1 mm
- net N$6: track 12.0 -> 13.8 mm
- net IO14: track 60.1 -> 58.5 mm
Other:
- board text added: "3.3V"
- board text added: "5V"
- board text added: "Alarm Clock"
- board text added: "GND"
- board text added: "RX"
- board text added: "TX"
- board text added: "V 1.0"

Commit message: Add files via upload
Parts:
- T1: value BC848 -> BC817-25LT1SMD; device transistor:SOT23 -> transistor-npn:SOT23-BEC
Connections:
- net GND: now also T1.E; no longer T1.2
- net N$1: now also T1.C; no longer T1.3
- net N$7: now also T1.B; no longer T1.1
Changed lines of the file:
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@@
 <attribute name="VALUE" x="12.175" y="56.38" size="1.27" layer="27" rot="R90"/>
 </element>
-<element name="T1" library="transistor" library_urn="urn:adsk.eagle:library:402" package="SOT23" package3d_urn="urn:adsk.eagle:package:28738/2" value="BC848" x="60" y="16" smashed="yes" rot="R270">
+<element name="T1" library="transistor-npn" library_urn="urn:adsk.eagle:library:398" package="SOT23-BEC" package3d_urn="urn:adsk.eagle:package:28748/2" value="BC817-25LT1SMD" x="60" y="16" smashed="yes" rot="R270">
 <attribute name="NAME" x="58.895" y="17.705" size="1.27" layer="25"/>
 <attribute name="POPULARITY" value="0" x="60" y="16" size="1.778" layer="27" rot="R270" display="off"/>
@@
 <via x="66" y="38" extent="1-16" drill="0.35"/>
 <contactref element="BME280" pad="5"/>
-<contactref element="T1" pad="2"/>
+<contactref element="T1" pad="E"/>
 <contactref element="BTN" pad="1"/>
 <via x="72" y="53" extent="1-16" drill="0.35"/>
+<wire x1="72" y1="53" x2="81.3" y2="52.95" width="0" layer="19" extent="1-1"/>
+<wire x1="63.3" y1="52.95" x2="72" y2="53" width="0" layer="19" extent="1-1"/>
+<wire x1="58" y1="60.35" x2="63.3" y2="52.95" width="0" layer="19" extent="1-1"/>
+<wire x1="53" y1="60.35" x2="58" y2="60.35" width="0" layer="19" extent="1-1"/>
+<wire x1="48" y1="60.4" x2="53" y2="60.35" width="0" layer="19" extent="1-1"/>
+<wire x1="43" y1="60.4" x2="48" y2="60.4" width="0" layer="19" extent="1-1"/>
+<wire x1="49.32" y1="65.92" x2="48" y2="60.4" width="0" layer="19" extent="1-1"/>
+<wire x1="58" y1="70.45" x2="49.32" y2="65.92" width="0" layer="19" extent="1-1"/>
+<wire x1="63.02" y1="70.432" x2="58" y2="70.45" width="0" layer="19" extent="1-1"/>
+<wire x1="58" y1="44.6" x2="63.3" y2="52.95" width="0" layer="19" extent="1-1"/>
+<wire x1="66" y1="38" x2="58" y2="44.6" width="0" layer="19" extent="1-1"/>
+<wire x1="66.585" y1="34.95" x2="66" y2="38" width="0" layer="19" extent="1-1"/>
+<wire x1="31.93" y1="62.71" x2="43" y2="60.4" width="0" layer="19" extent="1-1"/>
+<wire x1="31.27" y1="68" x2="31.93" y2="62.71" width="0" layer="19" extent="1-1"/>
+<wire x1="58.9" y1="15.05" x2="66.585" y2="34.95" width="0" layer="19" extent="1-1"/>
+<wire x1="9" y1="67.81" x2="31.27" y2="68" width="0" layer="19" extent="1-1"/>
+<wire x1="90.31" y1="15.61" x2="66.585" y2="34.95" width="0" layer="19" extent="1-1"/>
+<wire x1="6.37" y1="19.9" x2="9" y2="67.81" width="0" layer="19" extent="1-1"/>
 </signal>
 <signal name="VDD">
@@
 </signal>
 <signal name="N$7">
-<contactref element="T1" pad="1"/>
+<contactref element="T1" pad="B"/>
 <contactref element="R1" pad="2"/>
 <wire x1="59" y1="20.578" x2="59" y2="17.05" width="0.508" layer="1"/>
@@
 <signal name="N$1">
 <contactref element="SG1" pad="-"/>
-<contactref element="T1" pad="3"/>
+<contactref element="T1" pad="C"/>
 <wire x1="61.1" y1="16" x2="61.2" y2="15.9" width="0.508" layer="1"/>
 <wire x1="67.99" y1="15.9" x2="61.2" y2="15.9" width="0.508" layer="1"/>

Commit message: Add files via upload
Parts:
- added BOOT: (no value), rcl:R1206
- added C5: 0,1uF, rcl:C1206
- moved RST 36.5 mm to (27.0, 63.0), turned to 0 degrees
- moved BTN 5.10 mm to (25.0, 69.0)
Connections:
- net EN: now also C5.2, RST.2
- net GND: now also BOOT.2, C5.1, RST.1; no longer RST.2
- net IO0: now also BOOT.1; no longer RST.1
Routing:
- net EN: track 8.52 -> 49.5 mm
- net IO35: track 58.0 -> 61.1 mm
Changed lines of the file:
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@@
 <element name="C1" library="rcl" library_urn="urn:adsk.eagle:library:334" package="C1206" package3d_urn="urn:adsk.eagle:package:23618/2" value="0,1uF" x="58" y="69.05" smashed="yes" rot="R270">
 <attribute name="NAME" x="56.88" y="71.67" size="1.27" layer="25"/>
-<attribute name="POPULARITY" value="54" x="-5.5" y="37.3" size="1.778" layer="27" rot="R270" display="off"/>
 <attribute name="SPICEPREFIX" value="C" x="-5.5" y="37.3" size="1.778" layer="27" rot="R270" display="off"/>
 </element>
 <element name="C2" library="rcl" library_urn="urn:adsk.eagle:library:334" package="C1206" package3d_urn="urn:adsk.eagle:package:23618/2" value="0,1uF" x="58" y="46" smashed="yes" rot="R90">
 <attribute name="NAME" x="59.17" y="43.43" size="1.27" layer="25" rot="R180"/>
-<attribute name="POPULARITY" value="54" x="121.5" y="84.1" size="1.778" layer="27" rot="R90" display="off"/>
 <attribute name="SPICEPREFIX" value="C" x="121.5" y="84.1" size="1.778" layer="27" rot="R90" display="off"/>
 </element>
 <element name="C3" library="rcl" library_urn="urn:adsk.eagle:library:334" package="C1206" package3d_urn="urn:adsk.eagle:package:23618/2" value="10uF" x="53" y="58.95" smashed="yes" rot="R270">
 <attribute name="NAME" x="54.12" y="56.43" size="1.27" layer="25" rot="R180"/>
-<attribute name="POPULARITY" value="54" x="-10.5" y="1.8" size="1.778" layer="27" rot="R270" display="off"/>
 <attribute name="SPICEPREFIX" value="C" x="-10.5" y="1.8" size="1.778" layer="27" rot="R270" display="off"/>
 </element>
 <element name="C4" library="rcl" library_urn="urn:adsk.eagle:library:334" package="C1206" package3d_urn="urn:adsk.eagle:package:23618/2" value="0,1uF" x="58" y="58.95" smashed="yes" rot="R270">
 <attribute name="NAME" x="56.88" y="61.57" size="1.27" layer="25"/>
-<attribute name="POPULARITY" value="54" x="-5.5" y="14.5" size="1.778" layer="27" rot="R270" display="off"/>
 <attribute name="SPICEPREFIX" value="C" x="-5.5" y="14.5" size="1.778" layer="27" rot="R270" display="off"/>
 </element>
 <element name="C6" library="rcl" library_urn="urn:adsk.eagle:library:334" package="C1206" package3d_urn="urn:adsk.eagle:package:23618/2" value="0,1uF" x="43" y="59" smashed="yes" rot="R270">
 <attribute name="NAME" x="41.93" y="61.57" size="1.27" layer="25"/>
-<attribute name="POPULARITY" value="54" x="-20.5" y="8.2" size="1.778" layer="27" rot="R270" display="off"/>
 <attribute name="SPICEPREFIX" value="C" x="-20.5" y="8.2" size="1.778" layer="27" rot="R270" display="off"/>
 </element>
 <element name="C7" library="rcl" library_urn="urn:adsk.eagle:library:334" package="C1206" package3d_urn="urn:adsk.eagle:package:23618/2" value="10uF" x="48" y="59" smashed="yes" rot="R270">
 <attribute name="NAME" x="49.07" y="56.43" size="1.27" layer="25" rot="R180"/>
-<attribute name="POPULARITY" value="54" x="-15.5" y="-4.5" size="1.778" layer="27" rot="R270" display="off"/>
 <attribute name="SPICEPREFIX" value="C" x="-15.5" y="-4.5" size="1.778" layer="27" rot="R270" display="off"/>
 </element>
@@
 <attribute name="SPICEPREFIX" value="R" x="129.1" y="67.2" size="1.778" layer="27" rot="R90" display="off"/>
 </element>
-<element name="RST" library="rcl" library_urn="urn:adsk.eagle:library:334" package="R1206" package3d_urn="urn:adsk.eagle:package:23540/2" value="" x="63.02" y="69.01" smashed="yes" rot="R90">
-<attribute name="NAME" x="61.34" y="71.55" size="1.27" layer="25"/>
+<element name="BOOT" library="rcl" library_urn="urn:adsk.eagle:library:334" package="R1206" package3d_urn="urn:adsk.eagle:package:23540/2" value="" x="63.02" y="69.01" smashed="yes" rot="R90">
+<attribute name="NAME" x="60.44" y="71.55" size="1.27" layer="25"/>
 <attribute name="SPICEPREFIX" value="R" x="131.6" y="90.6" size="1.778" layer="27" rot="R90" display="off"/>
 <attribute name="VALUE" x="65.56" y="67.74" size="1.27" layer="27" rot="R90"/>
@@
 <attribute name="SPICEPREFIX" value="R" x="59" y="22" size="1.778" layer="27" rot="R270" display="off"/>
 </element>
-<element name="BTN" library="pinhead-ext" package="1X02" value="" x="30" y="68" smashed="yes" rot="R180">
-<attribute name="NAME" x="28.2838" y="69.8288" size="1.27" layer="25" ratio="10"/>
-<attribute name="VALUE" x="32.54" y="71.175" size="1.27" layer="27" rot="R180"/>
+<element name="BTN" library="pinhead-ext" package="1X02" value="" x="25" y="69" smashed="yes" rot="R180">
+<attribute name="NAME" x="23.2838" y="70.8288" size="1.27" layer="25" ratio="10"/>
+<attribute name="VALUE" x="27.54" y="72.175" size="1.27" layer="27" rot="R180"/>
+</element>
+<element name="C5" library="rcl" library_urn="urn:adsk.eagle:library:334" package="C1206" package3d_urn="urn:adsk.eagle:package:23618/2" value="0,1uF" x="27" y="58" smashed="yes">
+<attribute name="NAME" x="25.73" y="59.27" size="1.27" layer="25"/>
+<attribute name="SPICEPREFIX" value="C" x="16" y="70" size="1.778" layer="27" display="off"/>
+</element>
+<element name="RST" library="rcl" library_urn="urn:adsk.eagle:library:334" package="R1206" package3d_urn="urn:adsk.eagle:package:23540/2" value="" x="27" y="63" smashed="yes">
+<attribute name="NAME" x="25.43" y="64.27" size="1.27" layer="25"/>
+<attribute name="SPICEPREFIX" value="R" x="27" y="63" size="1.778" layer="27" display="off"/>
+<attribute name="VALUE" x="25.73" y="60.46" size="1.27" layer="27"/>
 </element>
 </elements>
@@
 <contactref element="IC1" pad="1"/>
 <contactref element="C1" pad="1"/>
-<contactref element="RST" pad="2"/>
+<contactref element="BOOT" pad="2"/>
 <contactref element="BT1" pad="P$2"/>
 <contactref element="SERIAL" pad="4"/>
@@
 <contactref element="BTN" pad="1"/>
 <via x="72" y="53" extent="1-16" drill="0.35"/>
-<wire x1="72" y1="53" x2="81.3" y2="52.95" width="0" layer="19" extent="1-1"/>
-<wire x1="63.3" y1="52.95" x2="72" y2="53" width="0" layer="19" extent="1-1"/>
-<wire x1="58" y1="60.35" x2="63.3" y2="52.95" width="0" layer="19" extent="1-1"/>
-<wire x1="53" y1="60.35" x2="58" y2="60.35" width="0" layer="19" extent="1-1"/>
-<wire x1="48" y1="60.4" x2="53" y2="60.35" width="0" layer="19" extent="1-1"/>
-<wire x1="43" y1="60.4" x2="48" y2="60.4" width="0" layer="19" extent="1-1"/>
-<wire x1="49.32" y1="65.92" x2="48" y2="60.4" width="0" layer="19" extent="1-1"/>
-<wire x1="58" y1="70.45" x2="49.32" y2="65.92" width="0" layer="19" extent="1-1"/>
-<wire x1="63.02" y1="70.432" x2="58" y2="70.45" width="0" layer="19" extent="1-1"/>
-<wire x1="58" y1="44.6" x2="63.3" y2="52.95" width="0" layer="19" extent="1-1"/>
-<wire x1="66" y1="38" x2="58" y2="44.6" width="0" layer="19" extent="1-1"/>
-<wire x1="66.585" y1="34.95" x2="66" y2="38" width="0" layer="19" extent="1-1"/>
-<wire x1="31.93" y1="62.71" x2="43" y2="60.4" width="0" layer="19" extent="1-1"/>
-<wire x1="31.27" y1="68" x2="31.93" y2="62.71" width="0" layer="19" extent="1-1"/>
-<wire x1="58.9" y1="15.05" x2="66.585" y2="34.95" width="0" layer="19" extent="1-1"/>
-<wire x1="9" y1="67.81" x2="31.27" y2="68" width="0" layer="19" extent="1-1"/>
-<wire x1="90.31" y1="15.61" x2="66.585" y2="34.95" width="0" layer="19" extent="1-1"/>
-<wire x1="6.37" y1="19.9" x2="9" y2="67.81" width="0" layer="19" extent="1-1"/>
+<contactref element="C5" pad="1"/>
+<contactref element="RST" pad="1"/>
 </signal>
 <signal name="VDD">
@@
 <wire x1="53.5" y1="64.8" x2="52.9" y2="64.2" width="0.6096" layer="1"/>
 <contactref element="BME280" pad="6"/>
-<wire x1="28.25" y1="71.6" x2="23" y2="66.35" width="0.6096" layer="1"/>
-<wire x1="23" y1="66.35" x2="14.2" y2="66.35" width="0.6096" layer="1"/>
-<wire x1="28.25" y1="71.6" x2="50.5" y2="71.6" width="0.6096" layer="1"/>
+<wire x1="23.25" y1="71.6" x2="18" y2="66.35" width="0.6096" layer="1"/>
+<wire x1="18" y1="66.35" x2="14.2" y2="66.35" width="0.6096" layer="1"/>
+<wire x1="23.25" y1="71.6" x2="50.5" y2="71.6" width="0.6096" layer="1"/>
 <wire x1="14.2" y1="66.35" x2="10.2" y2="70.35" width="0.6096" layer="1"/>
 <wire x1="10.2" y1="70.35" x2="9" y2="70.35" width="0.6096" layer="1"/>
@@
 <wire x1="57.98" y1="50.538" x2="58" y2="50.518" width="0.508" layer="1"/>
 <wire x1="58" y1="50.518" x2="58" y2="47.4" width="0.508" layer="1"/>
+<contactref element="C5" pad="2"/>
+<contactref element="RST" pad="2"/>
+<wire x1="28.422" y1="63" x2="28.422" y2="58.022" width="0.508" layer="1"/>
+<wire x1="28.422" y1="58.022" x2="28.4" y2="58" width="0.508" layer="1"/>
+<wire x1="28.4" y1="58" x2="41.4" y2="45" width="0.508" layer="1"/>
+<wire x1="55.6" y1="45" x2="58" y2="47.4" width="0.508" layer="1"/>
+<wire x1="41.4" y1="45" x2="55.6" y2="45" width="0.508" layer="1"/>
 </signal>
 <signal name="SENSOR_VP">
@@
 <wire x1="35.5" y1="42" x2="58.6" y2="42" width="0.508" layer="1"/>
 <wire x1="61.93" y1="45.33" x2="58.6" y2="42" width="0.508" layer="1"/>
-<wire x1="28.73" y1="68" x2="28.73" y2="48.77" width="0.508" layer="1"/>
-<wire x1="28.73" y1="48.77" x2="35.5" y2="42" width="0.508" layer="1"/>
+<wire x1="23.73" y1="69" x2="23.73" y2="53.77" width="0.508" layer="1"/>
+<wire x1="23.73" y1="53.77" x2="35.5" y2="42" width="0.508" layer="1"/>
 </signal>
 <signal name="IO26">
@@
 <contactref element="ESP32" pad="25"/>
 <contactref element="C1" pad="2"/>
-<contactref element="RST" pad="1"/>
+<contactref element="BOOT" pad="1"/>
 <wire x1="81.3" y1="36.44" x2="82.44" y2="36.44" width="0.508" layer="1"/>
 <wire x1="82.946" y1="36.946" x2="82.946" y2="47.35231875" width="0.508" layer="1"/>

Commit message: Add files via upload
Parts:
- moved R1 1.00 mm to (59.0, 23.0)
- flipped LCD to the top
Connections:
- net IO16: now also LCD.30
- net IO32: now also BTN.2; no longer BME280.4
- net IO33: now also BME280.4; no longer LCD.30
- net IO35: no longer BTN.2
Routing:
- net IO35: track 61.1 -> 0.00 mm
- net IO14: track 58.5 -> 29.4 mm, vias 0 -> 1
- net IO16: track 0.00 -> 20.7 mm, vias 0 -> 1
- net IO33: track 47.3 -> 65.6 mm
- net IO12: track 53.2 -> 64.2 mm
- net IO13: track 39.0 -> 49.1 mm
- net IO4: track 26.1 -> 32.7 mm
- net IO27: track 80.3 -> 74.3 mm
- net IO32: track 66.0 -> 60.5 mm
- net VDD: track 234.3 -> 229.6 mm
- net IO26: track 20.0 -> 18.7 mm
- net N$7: track 3.67 -> 4.67 mm

Commit message: Add files via upload
Routing:
- net IO16: track 20.7 -> 32.0 mm, vias 1 -> 0
- net IO2: track 26.2 -> 28.2 mm
- net IO15: track 27.2 -> 29.2 mm
- net IO4: track 32.7 -> 31.3 mm
Changed lines of the file:
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@@
 <wire x1="89.5" y1="52.4" x2="84.6" y2="47.5" width="0.508" layer="1"/>
 <wire x1="84.6" y1="47.5" x2="84.6" y2="35.6" width="0.508" layer="1"/>
-<wire x1="84.6" y1="35.6" x2="83.4" y2="34.4" width="0.508" layer="1"/>
-<wire x1="81.2" y1="37.61" x2="80.1" y2="37.61" width="0.508" layer="1"/>
+<wire x1="84.6" y1="35.6" x2="83.5" y2="34.5" width="0.508" layer="1"/>
+<wire x1="81.2" y1="37.61" x2="80.5" y2="37.61" width="0.508" layer="1"/>
 <wire x1="81.2" y1="37.61" x2="81.3" y2="37.71" width="0.508" layer="1"/>
-<wire x1="80.1652625" y1="34.4" x2="83.4" y2="34.4" width="0.508" layer="1"/>
-<wire x1="79.4" y1="36.91" x2="79.4" y2="35.1652625" width="0.508" layer="1"/>
-<wire x1="79.4" y1="35.1652625" x2="80.1652625" y2="34.4" width="0.508" layer="1"/>
-<wire x1="79.4" y1="36.91" x2="80.1" y2="37.61" width="0.508" layer="1"/>
+<wire x1="81.1652625" y1="34.5" x2="83.5" y2="34.5" width="0.508" layer="1"/>
+<wire x1="79.9" y1="37.01" x2="79.9" y2="35.7652625" width="0.508" layer="1"/>
+<wire x1="79.9" y1="35.7652625" x2="81.1652625" y2="34.5" width="0.508" layer="1"/>
+<wire x1="79.9" y1="37.01" x2="80.5" y2="37.61" width="0.508" layer="1"/>
 </signal>
 <signal name="IO0">
@@
 <wire x1="78.015" y1="34.95" x2="78.015" y2="34.015" width="0.508" layer="1"/>
 <wire x1="78.015" y1="34.015" x2="78" y2="34" width="0.508" layer="1"/>
-<wire x1="78" y1="34" x2="78.9396" y2="33.0604" width="0.508" layer="1"/>
-<wire x1="84.29435" y1="33.0604" x2="86.3396" y2="35.10565" width="0.508" layer="1"/>
+<wire x1="78" y1="34" x2="79.9396" y2="32.0604" width="0.508" layer="1"/>
+<wire x1="85.29435" y1="32.0604" x2="87.3396" y2="34.10565" width="0.508" layer="1"/>
 <wire x1="88.12603125" y1="44.7184" x2="91.4784" y2="44.7184" width="0.508" layer="1"/>
 <wire x1="91.4784" y1="44.7184" x2="92.85" y2="46.09" width="0.508" layer="1"/>
-<wire x1="86.3396" y1="35.10565" x2="86.3396" y2="42.93196875" width="0.508" layer="1"/>
-<wire x1="86.3396" y1="42.93196875" x2="88.12603125" y2="44.7184" width="0.508" layer="1"/>
-<wire x1="78.9396" y1="33.0604" x2="84.29435" y2="33.0604" width="0.508" layer="1"/>
+<wire x1="87.3396" y1="34.10565" x2="87.3396" y2="43.93196875" width="0.508" layer="1"/>
+<wire x1="87.3396" y1="43.93196875" x2="88.12603125" y2="44.7184" width="0.508" layer="1"/>
+<wire x1="79.9396" y1="32.0604" x2="85.29435" y2="32.0604" width="0.508" layer="1"/>
 </signal>
 <signal name="IO15">
@@
 <contactref element="LCD" pad="23"/>
 <wire x1="76.745" y1="34.95" x2="76.745" y2="33.255" width="0.508" layer="1"/>
-<wire x1="76.745" y1="33.255" x2="78.3" y2="31.7" width="0.508" layer="1"/>
-<wire x1="78.3" y1="31.7" x2="85" y2="31.7" width="0.508" layer="1"/>
-<wire x1="87.6" y1="34.3" x2="87.6" y2="40.8" width="0.508" layer="1"/>
-<wire x1="87.6" y1="40.8" x2="89.0816" y2="42.2816" width="0.508" layer="1"/>
+<wire x1="76.745" y1="33.255" x2="79.3" y2="30.7" width="0.508" layer="1"/>
+<wire x1="79.3" y1="30.7" x2="86" y2="30.7" width="0.508" layer="1"/>
+<wire x1="88.6" y1="33.3" x2="88.6" y2="41.8" width="0.508" layer="1"/>
+<wire x1="88.6" y1="41.8" x2="89.0816" y2="42.2816" width="0.508" layer="1"/>
 <wire x1="89.0816" y1="42.2816" x2="91.59396875" y2="42.2816" width="0.508" layer="1"/>
 <wire x1="92.85" y1="43.55" x2="92.85" y2="43.53763125" width="0.508" layer="1"/>
 <wire x1="92.85" y1="43.53763125" x2="91.59396875" y2="42.2816" width="0.508" layer="1"/>
-<wire x1="85" y1="31.7" x2="87.6" y2="34.3" width="0.508" layer="1"/>
+<wire x1="86" y1="30.7" x2="88.6" y2="33.3" width="0.508" layer="1"/>
 </signal>
 <signal name="SD1">
@@
 <contactref element="LCD" pad="30"/>
 <wire x1="90.31" y1="51.17" x2="90.17" y2="51.17" width="0.508" layer="16"/>
-<wire x1="90.17" y1="51.17" x2="78" y2="39" width="0.508" layer="16"/>
-<via x="78" y="39" extent="1-16" drill="0.35"/>
-<wire x1="78" y1="39" x2="81.28" y2="39" width="0.508" layer="1"/>
 <wire x1="81.28" y1="39" x2="81.3" y2="38.98" width="0.508" layer="1"/>
+<wire x1="90.31" y1="51.17" x2="86" y2="46.86" width="0.508" layer="1"/>
+<wire x1="86" y1="46.86" x2="86" y2="35" width="0.508" layer="1"/>
+<wire x1="86" y1="35" x2="84.2" y2="33.2" width="0.508" layer="1"/>
+<wire x1="80.8" y1="33.2" x2="79.1" y2="34.9" width="0.508" layer="1"/>
+<wire x1="79.1" y1="34.9" x2="79.1" y2="37.7" width="0.508" layer="1"/>
+<wire x1="79.1" y1="37.7" x2="80.4" y2="39" width="0.508" layer="1"/>
+<wire x1="80.4" y1="39" x2="81.28" y2="39" width="0.508" layer="1"/>
+<wire x1="84.2" y1="33.2" x2="80.8" y2="33.2" width="0.508" layer="1"/>
 </signal>
 <signal name="IO27">
@@
 <contactref element="LCD" pad="31"/>
 <wire x1="63.3" y1="38.98" x2="62.28" y2="38.98" width="0.508" layer="1"/>
-<wire x1="62" y1="38.7" x2="62" y2="32" width="0.508" layer="1"/>
-<wire x1="62.28" y1="38.98" x2="62" y2="38.7" width="0.508" layer="1"/>
-<wire x1="62" y1="32" x2="69.5" y2="24.5" width="0.508" layer="1"/>
+<wire x1="61.6" y1="38.3" x2="61.6" y2="32.4" width="0.508" layer="1"/>
+<wire x1="62.28" y1="38.98" x2="61.6" y2="38.3" width="0.508" layer="1"/>
+<wire x1="61.6" y1="32.4" x2="69.5" y2="24.5" width="0.508" layer="1"/>
 <wire x1="93.5" y1="24.5" x2="96" y2="27" width="0.508" layer="1"/>
 <wire x1="96" y1="27" x2="96" y2="50.56" width="0.508" layer="1"/>

Commit message: Add files via upload
Parts:
- added R2, R3: 10k, rcl:R1206
- moved C5 3.61 mm to (29.0, 61.0), turned to 270 degrees
- moved RST 3.61 mm to (24.0, 61.0), turned to 270 degrees
- moved BTN 1.00 mm to (25.0, 68.0)
Connections:
- net GND: now also R3.1
- net IO35: now also R2.1, R3.2
- net VIN: now also R2.2
Routing:
- net IO35: track 0.00 -> 72.7 mm
- net IO32: track 60.5 -> 63.6 mm
- net VIN: track 57.1 -> 59.7 mm
- net EN: track 49.5 -> 51.5 mm
- net IO25: track 65.4 -> 66.3 mm
- net IO33: track 65.6 -> 66.4 mm
- net VDD: track 229.6 -> 230.3 mm
