File: AlarmClock.sch (EAGLE design)
At the start: 20 parts, among them IC1 LD1117AS33TR, T1 BC848

Commit message: Add files via upload
Parts:
- R1: value (none) -> 10k
Changed lines of the file:
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@@
 <part name="VDD1" library="supply1" library_urn="urn:adsk.eagle:library:371" deviceset="VDD" device=""/>
 <part name="T1" library="transistor" library_urn="urn:adsk.eagle:library:402" deviceset="BC848" device="" package3d_urn="urn:adsk.eagle:package:28738/2"/>
-<part name="R1" library="rcl" library_urn="urn:adsk.eagle:library:334" deviceset="R-EU_" device="R1206" package3d_urn="urn:adsk.eagle:package:23540/2"/>
+<part name="R1" library="rcl" library_urn="urn:adsk.eagle:library:334" deviceset="R-EU_" device="R1206" package3d_urn="urn:adsk.eagle:package:23540/2" value="10k"/>
 <part name="GND8" library="supply1" library_urn="urn:adsk.eagle:library:371" deviceset="GND" device=""/>
 <part name="VDD5" library="supply1" library_urn="urn:adsk.eagle:library:371" deviceset="VDD" device=""/>
 <part name="GND5" library="supply1" library_urn="urn:adsk.eagle:library:371" deviceset="GND" device=""/>
 <part name="JP1" library="pinhead-ext" deviceset="PINHD-1X2" device="_2.54"/>
+<part name="VDD6" library="supply1" library_urn="urn:adsk.eagle:library:371" deviceset="VDD" device=""/>
 </parts>
 <sheets>
@@
 </instance>
 <instance part="SG1" gate="G$1" x="195.58" y="149.86" smashed="yes" rot="R90">
-<attribute name="NAME" x="189.23" y="147.32" size="1.778" layer="95" rot="R90"/>
+<attribute name="NAME" x="185.42" y="151.13" size="1.778" layer="95"/>
 </instance>
 <instance part="BME280" gate="A" x="101.6" y="25.4" smashed="yes" rot="R180">
@@
 </instance>
 <instance part="T1" gate="G$1" x="195.58" y="132.08" smashed="yes">
-<attribute name="NAME" x="185.42" y="139.7" size="1.778" layer="95"/>
-<attribute name="VALUE" x="185.42" y="137.16" size="1.778" layer="96"/>
+<attribute name="NAME" x="195.58" y="134.62" size="1.778" layer="95"/>
+<attribute name="VALUE" x="198.12" y="129.54" size="1.778" layer="96"/>
 </instance>
 <instance part="R1" gate="G$1" x="187.96" y="132.08" smashed="yes">
 <attribute name="NAME" x="186.1566" y="133.35" size="1.778" layer="95"/>
-<attribute name="VALUE" x="185.928" y="131.064" size="1.778" layer="96" rot="R270"/>
+<attribute name="VALUE" x="186.182" y="129.032" size="1.778" layer="96"/>
 </instance>
 <instance part="GND8" gate="1" x="198.12" y="124.46" smashed="yes">
@@
 <attribute name="NAME" x="115.57" y="73.025" size="1.778" layer="95" rot="R180"/>
 <attribute name="VALUE" x="115.57" y="83.82" size="1.778" layer="96" rot="R180"/>
+</instance>
+<instance part="VDD6" gate="G$1" x="53.34" y="27.94" smashed="yes">
+<attribute name="VALUE" x="50.8" y="30.48" size="1.778" layer="96"/>
 </instance>
 </instances>
@@
 <pinref part="LCD" gate="A" pin="2"/>
 <wire x1="41.91" y1="25.4" x2="53.34" y2="25.4" width="0.1524" layer="91"/>
-<label x="48.26" y="25.4" size="1.778" layer="95"/>
-</segment>
-<segment>
+<pinref part="VDD6" gate="G$1" pin="VDD"/>
+</segment>
+<segment>

Commit message: Add files via upload
Parts:
- renumbered JP1 to BTN
Connections:
- net IO25: now also BME280.3
- net IO26: now also R1.1
- net IO27: now also LCD.31
- net IO32: now also BME280.4; no longer LCD.31
- net IO34: no longer BME280.3
- net IO35: now also BTN.2; no longer R1.1
- net SENSOR_VN: no longer BME280.4
- net SENSOR_VP: no longer BTN.2
Changed lines of the file:
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@@
 <part name="VDD5" library="supply1" library_urn="urn:adsk.eagle:library:371" deviceset="VDD" device=""/>
 <part name="GND5" library="supply1" library_urn="urn:adsk.eagle:library:371" deviceset="GND" device=""/>
-<part name="JP1" library="pinhead-ext" deviceset="PINHD-1X2" device="_2.54"/>
+<part name="BTN" library="pinhead-ext" deviceset="PINHD-1X2" device="_2.54"/>
 <part name="VDD6" library="supply1" library_urn="urn:adsk.eagle:library:371" deviceset="VDD" device=""/>
 </parts>
@@
 <attribute name="VALUE" x="119.38" y="71.12" size="1.778" layer="96"/>
 </instance>
-<instance part="JP1" gate="G$1" x="109.22" y="78.74" smashed="yes" rot="R180">
-<attribute name="NAME" x="115.57" y="73.025" size="1.778" layer="95" rot="R180"/>
+<instance part="BTN" gate="G$1" x="109.22" y="78.74" smashed="yes" rot="R180">
+<attribute name="NAME" x="107.95" y="81.915" size="1.778" layer="95"/>
 <attribute name="VALUE" x="115.57" y="83.82" size="1.778" layer="96" rot="R180"/>
 </instance>
@@
 </segment>
 <segment>
-<pinref part="JP1" gate="G$1" pin="1"/>
+<pinref part="BTN" gate="G$1" pin="1"/>
 <pinref part="GND5" gate="1" pin="GND"/>
 <wire x1="121.92" y1="76.2" x2="111.76" y2="76.2" width="0.1524" layer="91"/>
@@
 <label x="43.18" y="152.4" size="1.778" layer="95"/>
 </segment>
-<segment>
-<wire x1="111.76" y1="78.74" x2="121.92" y2="78.74" width="0.1524" layer="91"/>
-<pinref part="JP1" gate="G$1" pin="2"/>
-<label x="116.84" y="78.74" size="1.778" layer="95"/>
-</segment>
 </net>
 <net name="SENSOR_VN" class="0">
@@
 <label x="43.18" y="149.86" size="1.778" layer="95"/>
 </segment>
-<segment>
-<wire x1="104.14" y1="25.4" x2="114.3" y2="25.4" width="0.1524" layer="91"/>
-<pinref part="BME280" gate="A" pin="4"/>
-<label x="109.22" y="25.4" size="1.778" layer="95"/>
-</segment>
 </net>
 <net name="IO34" class="0">
@@
 <label x="43.18" y="147.32" size="1.778" layer="95"/>
 </segment>
-<segment>
-<pinref part="BME280" gate="A" pin="3"/>
-<wire x1="104.14" y1="22.86" x2="114.3" y2="22.86" width="0.1524" layer="91"/>
-<label x="109.22" y="22.86" size="1.778" layer="95"/>
-</segment>
 </net>
 <net name="IO35" class="0">
@@
 </segment>
 <segment>
-<pinref part="R1" gate="G$1" pin="1"/>
-<wire x1="182.88" y1="132.08" x2="172.72" y2="132.08" width="0.1524" layer="91"/>
-<label x="172.72" y="132.08" size="1.778" layer="95"/>
+<pinref part="BTN" gate="G$1" pin="2"/>
+<wire x1="111.76" y1="78.74" x2="121.92" y2="78.74" width="0.1524" layer="91"/>
+<label x="116.84" y="78.74" size="1.778" layer="95"/>
 </segment>
 </net>
@@
 <pinref part="ESP32" gate="G$1" pin="IO26"/>
 <label x="43.18" y="134.62" size="1.778" layer="95"/>
+</segment>
+<segment>
+<pinref part="R1" gate="G$1" pin="1"/>
+<wire x1="182.88" y1="132.08" x2="170.18" y2="132.08" width="0.1524" layer="91"/>
+<label x="170.18" y="132.08" size="1.778" layer="95"/>
 </segment>
 </net>
@@
 </segment>
 <segment>
+<pinref part="BME280" gate="A" pin="4"/>
+<wire x1="104.14" y1="25.4" x2="114.3" y2="25.4" width="0.1524" layer="91"/>
+<label x="109.22" y="25.4" size="1.778" layer="95"/>
+</segment>
+</net>
+<net name="IO33" class="0">
+<segment>
+<wire x1="58.42" y1="139.7" x2="43.18" y2="139.7" width="0.1524" layer="91"/>
+<pinref part="ESP32" gate="G$1" pin="IO33"/>
+<label x="43.18" y="139.7" size="1.778" layer="95"/>
+</segment>
+<segment>
+<wire x1="41.91" y1="60.96" x2="53.34" y2="60.96" width="0.1524" layer="91"/>
+<pinref part="LCD" gate="A" pin="30"/>
+<label x="48.26" y="60.96" size="1.778" layer="95"/>
+</segment>
+</net>
+<net name="IO25" class="0">
+<segment>
+<wire x1="58.42" y1="137.16" x2="43.18" y2="137.16" width="0.1524" layer="91"/>
+<pinref part="ESP32" gate="G$1" pin="IO25"/>
+<label x="43.18" y="137.16" size="1.778" layer="95"/>
+</segment>
+<segment>
+<pinref part="BME280" gate="A" pin="3"/>
+<wire x1="104.14" y1="22.86" x2="114.3" y2="22.86" width="0.1524" layer="91"/>
+<label x="109.22" y="22.86" size="1.778" layer="95"/>
+</segment>
+</net>
+<net name="N$5" class="0">
+<segment>
+<pinref part="BT2" gate="G$1" pin="+"/>
+<pinref part="BT3" gate="G$1" pin="-"/>
+</segment>
+</net>
+<net name="N$6" class="0">
+<segment>
+<pinref part="BT1" gate="G$1" pin="-"/>
+<pinref part="BT3" gate="G$1" pin="+"/>
+</segment>
+</net>
+<net name="IO18" class="0">
+<segment>
+<pinref part="ESP32" gate="G$1" pin="IO18"/>
+<wire x1="106.68" y1="139.7" x2="119.38" y2="139.7" width="0.1524" layer="91"/>
+<label x="114.3" y="139.7" size="1.778" layer="95"/>
+</segment>
+</net>
+<net name="IO21" class="0">
+<segment>
+<wire x1="119.38" y1="147.32" x2="106.68" y2="147.32" width="0.1524" layer="91"/>
+<pinref part="ESP32" gate="G$1" pin="IO21"/>
+<label x="114.3" y="147.32" size="1.778" layer="95"/>
+</segment>
+</net>
+<net name="IO19" class="0">
+<segment>
+<pinref part="ESP32" gate="G$1" pin="IO19"/>
+<wire x1="106.68" y1="142.24" x2="119.38" y2="142.24" width="0.1524" layer="91"/>
+<label x="114.3" y="142.24" size="1.778" layer="95"/>
+</segment>
+</net>
+<net name="IO5" class="0">
+<segment>
+<pinref part="ESP32" gate="G$1" pin="IO5"/>
+<wire x1="106.68" y1="137.16" x2="119.38" y2="137.16" width="0.1524" layer="91"/>
+<label x="114.3" y="137.16" size="1.778" layer="95"/>
+</segment>
+</net>
+<net name="IO17" class="0">
+<segment>
+<pinref part="ESP32" gate="G$1" pin="IO17"/>
+<wire x1="106.68" y1="134.62" x2="119.38" y2="134.62" width="0.1524" layer="91"/>
+<label x="114.3" y="134.62" size="1.778" layer="95"/>
+</segment>
+</net>
+<net name="IO16" class="0">
+<segment>
+<pinref part="ESP32" gate="G$1" pin="IO16"/>
+<wire x1="106.68" y1="132.08" x2="119.38" y2="132.08" width="0.1524" layer="91"/>
+<label x="114.3" y="132.08" size="1.778" layer="95"/>
+</segment>
+</net>
+<net name="IO27" class="0">
+<segment>
+<wire x1="58.42" y1="132.08" x2="43.18" y2="132.08" width="0.1524" layer="91"/>
+<pinref part="ESP32" gate="G$1" pin="IO27"/>
+<label x="43.18" y="132.08" size="1.778" layer="95"/>
+</segment>
+<segment>
 <pinref part="LCD" gate="A" pin="31"/>
 <wire x1="34.29" y1="63.5" x2="20.32" y2="63.5" width="0.1524" layer="91"/>
@@
 </segment>
 </net>
-<net name="IO33" class="0">
-<segment>
-<wire x1="58.42" y1="139.7" x2="43.18" y2="139.7" width="0.1524" layer="91"/>
-<pinref part="ESP32" gate="G$1" pin="IO33"/>
-<label x="43.18" y="139.7" size="1.778" layer="95"/>
-</segment>
-<segment>
-<wire x1="41.91" y1="60.96" x2="53.34" y2="60.96" width="0.1524" layer="91"/>
-<pinref part="LCD" gate="A" pin="30"/>
-<label x="48.26" y="60.96" size="1.778" layer="95"/>
-</segment>
-</net>
-<net name="IO25" class="0">
-<segment>
-<wire x1="58.42" y1="137.16" x2="43.18" y2="137.16" width="0.1524" layer="91"/>
-<pinref part="ESP32" gate="G$1" pin="IO25"/>
-<label x="43.18" y="137.16" size="1.778" layer="95"/>
-</segment>
-</net>
-<net name="N$5" class="0">
-<segment>
-<pinref part="BT2" gate="G$1" pin="+"/>
-<pinref part="BT3" gate="G$1" pin="-"/>
-</segment>
-</net>
-<net name="N$6" class="0">
-<segment>
-<pinref part="BT1" gate="G$1" pin="-"/>
-<pinref part="BT3" gate="G$1" pin="+"/>
-</segment>
-</net>
-<net name="IO18" class="0">
-<segment>
-<pinref part="ESP32" gate="G$1" pin="IO18"/>
-<wire x1="106.68" y1="139.7" x2="119.38" y2="139.7" width="0.1524" layer="91"/>
-<label x="114.3" y="139.7" size="1.778" layer="95"/>
-</segment>
-</net>
-<net name="IO21" class="0">
-<segment>
-<wire x1="119.38" y1="147.32" x2="106.68" y2="147.32" width="0.1524" layer="91"/>
-<pinref part="ESP32" gate="G$1" pin="IO21"/>
-<label x="114.3" y="147.32" size="1.778" layer="95"/>
-</segment>
-</net>
-<net name="IO19" class="0">
-<segment>
-<pinref part="ESP32" gate="G$1" pin="IO19"/>
-<wire x1="106.68" y1="142.24" x2="119.38" y2="142.24" width="0.1524" layer="91"/>
-<label x="114.3" y="142.24" size="1.778" layer="95"/>
-</segment>
-</net>
-<net name="IO5" class="0">
-<segment>
-<pinref part="ESP32" gate="G$1" pin="IO5"/>
-<wire x1="106.68" y1="137.16" x2="119.38" y2="137.16" width="0.1524" layer="91"/>
-<label x="114.3" y="137.16" size="1.778" layer="95"/>
-</segment>
-</net>
-<net name="IO17" class="0">
-<segment>
-<pinref part="ESP32" gate="G$1" pin="IO17"/>
-<wire x1="106.68" y1="134.62" x2="119.38" y2="134.62" width="0.1524" layer="91"/>
-<label x="114.3" y="134.62" size="1.778" layer="95"/>
-</segment>
-</net>
-<net name="IO16" class="0">
-<segment>
-<pinref part="ESP32" gate="G$1" pin="IO16"/>
-<wire x1="106.68" y1="132.08" x2="119.38" y2="132.08" width="0.1524" layer="91"/>
-<label x="114.3" y="132.08" size="1.778" layer="95"/>
-</segment>
-</net>
-<net name="IO27" class="0">
-<segment>
-<wire x1="58.42" y1="132.08" x2="43.18" y2="132.08" width="0.1524" layer="91"/>
-<pinref part="ESP32" gate="G$1" pin="IO27"/>
-<label x="43.18" y="132.08" size="1.778" layer="95"/>
-</segment>
-</net>

Commit message: Add files via upload
Parts:
- BT1, BT2, BT3: value (none) -> HALTER1XUM4-LF; device SparkFun-Batteries:BATTERY-AAA -> TheLibrary:HALTER1XUM4-LF
Connections:
- removed net N$6 (its old number): BT1.-, BT3.+
- new net N$5: BT1.+, BT2.-
- net GND: now also BT1.-; no longer BT2.-
- net VIN: now also BT3.+; no longer BT1.+
Other:
- moved on the sheet: BT1, BT2, BT3
Changed lines of the file:
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@@
 <part name="VDD3" library="supply1" library_urn="urn:adsk.eagle:library:371" deviceset="VDD" device=""/>
 <part name="VDD4" library="supply1" library_urn="urn:adsk.eagle:library:371" deviceset="VDD" device=""/>
-<part name="BT1" library="SparkFun-Batteries" deviceset="BATTERY" device="-AAA"/>
-<part name="BT2" library="SparkFun-Batteries" deviceset="BATTERY" device="-AAA"/>
+<part name="BT3" library="TheLibrary" deviceset="HALTER1XUM4-LF" device=""/>
+<part name="BT1" library="TheLibrary" deviceset="HALTER1XUM4-LF" device=""/>
 <part name="GND14" library="supply1" library_urn="urn:adsk.eagle:library:371" deviceset="GND" device=""/>
-<part name="BT3" library="SparkFun-Batteries" deviceset="BATTERY" device="-AAA"/>
+<part name="BT2" library="TheLibrary" deviceset="HALTER1XUM4-LF" device=""/>
 <part name="RST" library="rcl" library_urn="urn:adsk.eagle:library:334" deviceset="R-EU_" device="R1206" package3d_urn="urn:adsk.eagle:package:23540/2"/>
 <part name="SERIAL" library="pinhead-ext" deviceset="PINHD-1X5" device="_2.54-SMD-90°"/>
@@
 <attribute name="VALUE" x="238.76" y="72.39" size="1.778" layer="96"/>
 </instance>
-<instance part="BT1" gate="G$1" x="210.82" y="67.31" smashed="yes" rot="R180">
+<instance part="BT3" gate="G$1" x="210.82" y="67.31" smashed="yes" rot="R180">
 <attribute name="NAME" x="210.82" y="62.992" size="1.778" layer="95" font="vector" rot="R180" align="bottom-center"/>
 <attribute name="VALUE" x="210.82" y="71.628" size="1.778" layer="96" font="vector" rot="R180" align="top-center"/>
 </instance>
-<instance part="BT2" gate="G$1" x="190.5" y="67.31" smashed="yes" rot="R180">
+<instance part="BT1" gate="G$1" x="190.5" y="67.31" smashed="yes" rot="R180">
 <attribute name="NAME" x="190.5" y="62.992" size="1.778" layer="95" font="vector" rot="R180" align="bottom-center"/>
 <attribute name="VALUE" x="190.5" y="71.628" size="1.778" layer="96" font="vector" rot="R180" align="top-center"/>
@@
 <attribute name="VALUE" x="182.88" y="57.15" size="1.778" layer="96"/>
 </instance>
-<instance part="BT3" gate="G$1" x="200.66" y="67.31" smashed="yes" rot="R180">
+<instance part="BT2" gate="G$1" x="200.66" y="67.31" smashed="yes" rot="R180">
 <attribute name="NAME" x="200.66" y="62.992" size="1.778" layer="95" font="vector" rot="R180" align="bottom-center"/>
 <attribute name="VALUE" x="200.66" y="71.628" size="1.778" layer="96" font="vector" rot="R180" align="top-center"/>
@@
 <segment>
 <pinref part="GND14" gate="1" pin="GND"/>
-<pinref part="BT2" gate="G$1" pin="-"/>
+<pinref part="BT1" gate="G$1" pin="-"/>
 <wire x1="185.42" y1="62.23" x2="185.42" y2="67.31" width="0.1524" layer="91"/>
 </segment>
@@
 <pinref part="C6" gate="G$1" pin="2"/>
 <wire x1="223.52" y1="67.31" x2="220.98" y2="67.31" width="0.1524" layer="91"/>
-<pinref part="BT1" gate="G$1" pin="+"/>
+<pinref part="BT3" gate="G$1" pin="+"/>
 <wire x1="215.9" y1="67.31" x2="220.98" y2="67.31" width="0.1524" layer="91"/>
 <junction x="220.98" y="67.31"/>
@@
 <net name="N$5" class="0">
 <segment>
+<pinref part="BT1" gate="G$1" pin="+"/>
+<pinref part="BT2" gate="G$1" pin="-"/>
+</segment>
+</net>
+<net name="N$6" class="0">
+<segment>
+<pinref part="BT3" gate="G$1" pin="-"/>
 <pinref part="BT2" gate="G$1" pin="+"/>
-<pinref part="BT3" gate="G$1" pin="-"/>
-</segment>
-</net>
-<net name="N$6" class="0">
-<segment>
-<pinref part="BT1" gate="G$1" pin="-"/>
-<pinref part="BT3" gate="G$1" pin="+"/>
-</segment>
-</net>
+</segment>
+</net>

Commit message: Add files via upload
Parts:
- T1: value BC848 -> BC817-25LT1SMD; device transistor:BC848 -> transistor-npn:BC817-25LT1SMD
Changed lines of the file:
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@@
 <part name="GND7" library="SparkFun-PowerSymbols" deviceset="GND" device=""/>
 <part name="VDD1" library="supply1" library_urn="urn:adsk.eagle:library:371" deviceset="VDD" device=""/>
-<part name="T1" library="transistor" library_urn="urn:adsk.eagle:library:402" deviceset="BC848" device="" package3d_urn="urn:adsk.eagle:package:28738/2"/>
+<part name="T1" library="transistor-npn" library_urn="urn:adsk.eagle:library:398" deviceset="BC817*" device="SMD" package3d_urn="urn:adsk.eagle:package:28748/2" technology="-25LT1" value="BC817-25LT1SMD"/>
 <part name="R1" library="rcl" library_urn="urn:adsk.eagle:library:334" deviceset="R-EU_" device="R1206" package3d_urn="urn:adsk.eagle:package:23540/2" value="10k"/>
 <part name="GND8" library="supply1" library_urn="urn:adsk.eagle:library:371" deviceset="GND" device=""/>

Commit message: Add files via upload
Parts:
- added BOOT: (no value), rcl:R-EU_R1206
- added C5: 0,1uF, rcl:C-EUC1206
Connections:
- net EN: now also C5.2, RST.2
- net GND: now also BOOT.2, C5.1, RST.1; no longer RST.2
- net IO0: now also BOOT.1; no longer RST.1
Other:
- moved on the sheet: C1, C2, C3, C4, ESP32, R9, RST

Commit message: Add files via upload
Connections:
- net IO16: now also LCD.30
- net IO32: now also BTN.2; no longer BME280.4
- net IO33: now also BME280.4; no longer LCD.30
- net IO35: no longer BTN.2
Changed lines of the file:
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@@
 <label x="55.88" y="144.78" size="1.778" layer="95"/>
-</segment>
-<segment>
-<pinref part="BTN" gate="G$1" pin="2"/>
-<wire x1="111.76" y1="78.74" x2="121.92" y2="78.74" width="0.1524" layer="91"/>
-<label x="116.84" y="78.74" size="1.778" layer="95"/>
 </segment>
 </net>
@@
 </segment>
 <segment>
+<pinref part="BTN" gate="G$1" pin="2"/>
+<wire x1="111.76" y1="78.74" x2="121.92" y2="78.74" width="0.1524" layer="91"/>
+<label x="116.84" y="78.74" size="1.778" layer="95"/>
+</segment>
+</net>
+<net name="IO33" class="0">
+<segment>
+<wire x1="71.12" y1="139.7" x2="55.88" y2="139.7" width="0.1524" layer="91"/>
+<pinref part="ESP32" gate="G$1" pin="IO33"/>
+<label x="55.88" y="139.7" size="1.778" layer="95"/>
+</segment>
+<segment>
 <pinref part="BME280" gate="A" pin="4"/>
 <wire x1="104.14" y1="25.4" x2="114.3" y2="25.4" width="0.1524" layer="91"/>
@@
 </segment>
 </net>
-<net name="IO33" class="0">
-<segment>
-<wire x1="71.12" y1="139.7" x2="55.88" y2="139.7" width="0.1524" layer="91"/>
-<pinref part="ESP32" gate="G$1" pin="IO33"/>
-<label x="55.88" y="139.7" size="1.778" layer="95"/>
-</segment>
-<segment>
-<wire x1="41.91" y1="60.96" x2="53.34" y2="60.96" width="0.1524" layer="91"/>
-<pinref part="LCD" gate="A" pin="30"/>
-<label x="48.26" y="60.96" size="1.778" layer="95"/>
-</segment>
-</net>
 <net name="IO25" class="0">
 <segment>
@@
 <label x="127" y="132.08" size="1.778" layer="95"/>
 </segment>
-</net>
+<segment>
+<pinref part="LCD" gate="A" pin="30"/>
+<wire x1="41.91" y1="60.96" x2="53.34" y2="60.96" width="0.1524" layer="91"/>
+<label x="48.26" y="60.96" size="1.778" layer="95"/>
+</segment>
+</net>
